File: hardware/boost_manufacturing_rev_b/Boost converter/Boost converter.kicad_pcb (KiCad board)
At the start: 4 copper layers, 73 x 47 mm, 40 parts, among them J1 Conn_01x02_Socket, J2 Conn_01x02_Socket, Q1 CSD18540Q5B, Q2 CSD18540Q5B, U1 LM5122QMHX/NOPB

Commit message: hardware: refresh boost rev b outputs and add LM5050 OR-ing rev a package
Update Boost Converter Rev B design/manufacturing files and add a new LM5050 OR-ing manufacturing package with standardized documentation.

Boost Rev B:

- Updated KiCad source files (.kicad_sch/.kicad_pcb/.kicad_prl), symbol libraries, footprint library entries, and fp cache.

- Added MCU-controlled shutdown path by pulling LM5122 SS low via MOSFET.

- Kept UVLO path for threshold function (not used for shutdown), so each re-enable triggers a fresh soft-start ramp from SS release.

- Regenerated manufacturing artifacts: BOM, CPL, Gerbers, drill files, Gerber job, and Gerber.zip.

- Rotated project backup zips (removed older snapshots, added new snapshots).

- Updated Rev B README and bench test procedure to document SS-pull-down behavior and validation steps.

LM5050 OR-ing Rev A:

- Added new folder: hardware/lm5050_redundant_supply_manufacturing_rev_a following hardware naming conventions.

- Added KiCad project files, local libraries/footprints, BOM, CPL, Gerbers, Gerber.zip, and project backups for the High Side OR-ing board.

- Added standardized README and test_procedure_rev_a.md for bring-up and source switchover/reverse-blocking validation.

Repository docs and organization:

- Updated top-level README boost summary to include SS pull-down control and soft-start restart behavior.

- Moved rover software handoff doc to firmware/2026/rover-software-handoff.md and updated README references to the new path.
Parts:
- added J3: Conn_01x01_Pin, Connector_PinHeader_1.00mm:PinHeader_1x01_P1.00mm_Vertical, F.Cu at (157.0, 155.0)
- added MOSFET1: 2N7002, Boost_Converter_Footprint_Library:SOT-23TO-236_318-08_ONS, F.Cu at (162.0, 152.0)
- added R3: 100Ω, Resistor_SMD:R_0603_1608Metric, F.Cu at (159.8, 155.0)
- added R6: 160kΩ, Resistor_SMD:R_0603_1608Metric, F.Cu at (163.0, 155.0)
- L1: value 22uH -> 10uH
Routing:
- net /SS: track 2.28 -> 7.35 mm
- net Net-(MOSFET1-G): track 0.00 -> 3.69 mm
- net Net-(J3-Pin_1): track 0.00 -> 2.00 mm
- net GND: vias 388 -> 382
Other:
- board text added: "ON/OFF"
- board text added: "REV B Feb 11 2025"
- board text removed: "REV B Feb 8 2025"
